File: Kicad/Chat_Cartridge_V1.3/ZX_Cartridge.kicad_sch (KiCad schematic)
At the start: 21 parts, among them J1 Conn_01x05_Female, SW1 SW_Push, U1 GAL16V8, U2 74LS165, U3 mini_esp32, U4 74HC595, U5 5v module (hx1314G based), U7 27C512, U9 74HCT125

Commit message: New PCB and code
Small bug fixes in the code
Connections:
- net +3V3: no longer U4.10 (~{SRCLR}), U4.16 (VCC)
- net +5V: now also U4.10 (~{SRCLR}), U4.16 (VCC)
Changed lines of the file:
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@@
   (junction (at 239.014 16.256) (diameter 0) (color 0 0 0 0)
   )
+  (junction (at 218.694 109.22) (diameter 0) (color 0 0 0 0)
+  )
   (junction (at 161.798 77.47) (diameter 0) (color 0 0 0 0)
   )
@@
   (junction (at 277.114 34.29) (diameter 0) (color 0 0 0 0)
   )
-  (junction (at 213.614 109.22) (diameter 0) (color 0 0 0 0)
-  )
   (wire (pts (xy 158.242 69.85) (xy 167.386 69.85))
     (stroke (width 0) (type default) (color 0 0 0 0))
@@
     (stroke (width 0) (type default) (color 0 0 0 0))
   )
-  (wire (pts (xy 195.326 109.22) (xy 213.614 109.22))
+  (wire (pts (xy 195.326 109.22) (xy 218.694 109.22))
     (stroke (width 0) (type default) (color 0 0 0 0))
   )
@@
   )
   (wire (pts (xy 187.706 44.196) (xy 187.452 44.196))
-    (stroke (width 0) (type default) (color 0 0 0 0))
-  )
-  (wire (pts (xy 213.614 109.22) (xy 218.694 109.22))
     (stroke (width 0) (type default) (color 0 0 0 0))
   )
@@
     )
     (property "Datasheet" "" (id 3) (at 19.304 178.308 0)
-      (effects (font (size 1.27 1.27)) hide)
-    )
-    (pin "1")
-  )
-  (symbol (lib_id "power:+3.3V") (at 213.614 109.22 0) (unit 1)
-    (in_bom yes) (on_board yes) (fields_autoplaced)
-    (property "Reference" "#PWR?" (id 0) (at 213.614 113.03 0)
-      (effects (font (size 1.27 1.27)) hide)
-    )
-    (property "Value" "+3.3V" (id 1) (at 213.614 105.6442 0))
-    (property "Footprint" "" (id 2) (at 213.614 109.22 0)
-      (effects (font (size 1.27 1.27)) hide)
-    )
-    (property "Datasheet" "" (id 3) (at 213.614 109.22 0)
       (effects (font (size 1.27 1.27)) hide)
     )
@@
     (pin "1")
   )
+  (symbol (lib_id "power:+5V") (at 218.694 109.22 0) (unit 1)
+    (in_bom yes) (on_board yes) (fields_autoplaced)
+    (property "Reference" "#PWR0118" (id 0) (at 218.694 113.03 0)
+      (effects (font (size 1.27 1.27)) hide)
+    )
+    (property "Value" "+5V" (id 1) (at 218.694 105.6442 0))
+    (property "Footprint" "" (id 2) (at 218.694 109.22 0)
+      (effects (font (size 1.27 1.27)) hide)
+    )
+    (property "Datasheet" "" (id 3) (at 218.694 109.22 0)
+      (effects (font (size 1.27 1.27)) hide)
+    )
+    (pin "1")
+  )
   (symbol (lib_id "74xx:74HCT595") (at 195.326 128.524 0) (mirror y) (unit 1)
     (in_bom yes) (on_board yes)
@@
       (reference "#PWR0117") (unit 1) (value "+5V") (footprint "")
     )
+    (path "/cdeb183d-03ed-4334-82ba-8b5ca29564c5"
+      (reference "#PWR0118") (unit 1) (value "+5V") (footprint "")
+    )
     (path "/9ab97898-e56a-42b6-ad2d-dbc7fe9e8a94"
       (reference "#PWR0119") (unit 1) (value "GND") (footprint "")
@@
       (reference "#PWR0138") (unit 1) (value "+5V") (footprint "")
     )
-    (path "/76004765-6e34-42e5-bef2-e8d5daedc3a7"
-      (reference "#PWR?") (unit 1) (value "+3.3V") (footprint "")
-    )
     (path "/6cedd722-1c91-4397-afa3-9c519f3265bd"
