File: Kicad/Chat_Cartridge_V1.4/ZX_Cartridge.kicad_sch (KiCad schematic)
At the start: 27 parts, among them Q1 2N7000, Q2 2N7000, Q3 Q_PMOS_GDS, SW1 SW_Push, U1 GAL16V8, U2 74LS165, U3 mini_esp32, U4 74HC595, U5 5v module (hx1314G based), U7 27C512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

Commit message: small things
Parts:
- Q3: value Q_PMOS_GDS -> MMFT2955ET1
Other:
- moved on the sheet: Z1
