File: Kicad/Chat_Cartridge_V1.4/ZX_Cartridge.kicad_pcb (KiCad board)
At the start: 4 copper layers, 85.7 x 71.3 mm, 27 parts, among them Q1 2N7000, Q2 2N7000, Q3 Q_PMOS_GDS, SW1 SW_Push, U1 GAL16V8, U2 74LS165, U3 mini_esp32, U4 74HC595, U5 5v module (hx1314G based), U7 27C512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

Commit message: unstable
Parts:
- moved D2 1.93 mm to (73.3, 91.5)
- moved U5 1.72 mm to (77.9, 70.5)
Routing:
- net 12V out: track 43.1 -> 40.7 mm
- net A11: track 40.9 -> 39.5 mm
Changed lines of the file:
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@@
 		)
 		(property "Value" "1k5"
-			(at 7.69 -0.1 90)
+			(at 1.1275 1.952 90)
 			(layer "F.SilkS")
 			(effects
@@
 	(footprint "Diode_THT:D_DO-34_SOD68_P7.62mm_Horizontal"
 		(layer "F.Cu")
-		(at 73.3375 89.5985)
+		(at 73.3375 91.53)
 		(descr "Diode, DO-34_SOD68 series, Axial, Horizontal, pin pitch=7.62mm, length*diameter=3.04*1.6mm^2, https://www.nxp.com/docs/en/data-sheet/KTY83_SER.pdf")
 		(tags "Diode DO-34_SOD68 series Axial Horizontal pin pitch 7.62mm  length 3.04mm diameter 1.6mm")
@@
 		)
 		(property "Value" "BAT86"
-			(at 3.81 1.92 0)
+			(at -3.8475 -0.2185 0)
 			(layer "F.Fab")
 			(effects
@@
 		(tags "CMS SOT")
 		(property "Reference" "Q3"
-			(at 0 -4.5 0)
+			(at -5.72 -2.684 0)
 			(layer "F.SilkS")
 			(effects
@@
 	(footprint "Barts:5v_switching_TO220"
 		(layer "F.Cu")
-		(at 77.9 68.75 90)
+		(at 77.9 70.473 90)
 		(descr "Through hole straight socket strip, 1x03, 2.54mm pitch, single row (from Kicad 4.0.7), script generated")
 		(tags "Through hole socket strip THT 1x03 2.54mm single row")
@@
 	)
 	(segment
-		(start 76.9 78.26)
-		(end 76.9 71.55)
+		(start 79.375 96.774)
+		(end 76.25 96.774)
 		(width 0.5)
 		(layer "F.Cu")
@@
 	)
 	(segment
-		(start 78.949 80.309)
-		(end 76.9 78.26)
+		(start 76.9 70.838)
+		(end 77.878 69.86)
 		(width 0.5)
 		(layer "F.Cu")
@@
 	)
 	(segment
-		(start 79.375 89.535)
+		(start 79.375 91.55)
 		(end 79.375 80.735)
 		(width 0.5)
@@
 	)
 	(segment
-		(start 79.375 96.774)
-		(end 76.25 96.774)
-		(width 0.5)
-		(layer "F.Cu")
-		(net 6)
-	)
-	(segment
-		(start 76.9 71.55)
-		(end 77.878 70.572)
-		(width 0.5)
-		(layer "F.Cu")
-		(net 6)
-	)
-	(segment
 		(start 79.375 80.735)
-		(end 78.949 80.309)
+		(end 76.9 78.26)
 		(width 0.5)
 		(layer "F.Cu")
@@
 	)
 	(segment
-		(start 77.878 70.572)
-		(end 77.878 68.137)
+		(start 79.375 91.55)
+		(end 79.355 91.53)
 		(width 0.5)
 		(layer "F.Cu")
@@
 	)
 	(segment
-		(start 79.375 89.535)
-		(end 79.3115 89.5985)
+		(start 76.9 78.26)
+		(end 76.9 70.838)
 		(width 0.5)
 		(layer "F.Cu")
@@
 	(segment
 		(start 79.375 96.774)
-		(end 79.375 89.535)
+		(end 79.375 91.55)
 		(width 0.5)
 		(layer "F.Cu")
@@
 	)
 	(segment
-		(start 79.3115 89.5985)
-		(end 73.3375 89.5985)
+		(start 79.355 91.53)
+		(end 73.3375 91.53)
 		(width 0.5)
 		(layer "F.Cu")
@@
 	)
 	(segment
-		(start 73.35 89.5)
-		(end 73.35 90.11)
-		(width 0.6)
-		(layer "In1.Cu")
-		(net 6)
-	)
-	(segment
-		(start 73.39 89.46)
-		(end 73.35 89.5)
-		(width 0.6)
-		(layer "In1.Cu")
-		(net 6)
-	)
-	(segment
 		(start 75.858 94.742)
 		(end 75.844 94.756)
@@
 	)
 	(segment
-		(start 73.35 70.85)
-		(end 73.35 70.75)
-		(width 0.6)
-		(layer "In1.Cu")
-		(net 25)
-	)
-	(segment
-		(start 73.35 70.75)
-		(end 72.798 70.198)
+		(start 86.15 112.09)
+		(end 88.65 109.59)
 		(width 0.6)
 		(layer "In1.Cu")
@@
 	)
 	(segment
-		(start 86.15 112.09)
-		(end 88.65 109.59)
+		(start 73.35 87.21)
+		(end 75.79 89.65)
 		(width 0.6)
 		(layer "In1.Cu")
@@
 	)
 	(segment
-		(start 71.4375 91.059)
-		(end 71.4375 88.082)
+		(start 72.798 70.198)
+		(end 73.35 70.75)
 		(width 0.6)
 		(layer "In1.Cu")
@@
 	)
 	(segment
-		(start 73.8055 66.4845)
-		(end 83.5655 66.4845)
-		(width 0.6)
-		(layer "In1.Cu")
-		(net 25)
-	)
-	(segment
 		(start 73.38 112.09)
 		(end 73.38 114.52)
@@
 	)
 	(segment
-		(start 72.798 67.027)
-		(end 73.3405 66.4845)
-		(width 0.6)
-		(layer "In1.Cu")
-		(net 25)
-	)
-	(segment
 		(start 68.78 114.6)
 		(end 73.3 114.6)
@@
 	)
 	(segment
+		(start 83.5655 66.4845)
+		(end 73.3405 66.4845)
+		(width 0.6)
+		(layer "In1.Cu")
+		(net 25)
+	)
+	(segment
 		(start 82.3595 74.2365)
 		(end 84.353 72.243)
@@
 	)
 	(segment
-		(start 73.3405 66.4845)
-		(end 73.8055 66.4845)
+		(start 73.38 112.09)
+		(end 73.35 112.12)
 		(width 0.6)
 		(layer "In1.Cu")
@@
 	)
 	(segment
-		(start 73.38 112.09)
-		(end 73.35 112.12)
+		(start 73.35 70.75)
+		(end 73.35 87.21)
 		(width 0.6)
 		(layer "In1.Cu")
@@
 	)
 	(segment
-		(start 107.975 68.7)
-		(end 107.975 68.725)
+		(start 75.79 89.65)
+		(end 75.79 93.49)
 		(width 0.6)
 		(layer "In1.Cu")
@@
 	)
 	(segment
-		(start 71.4375 88.082)
-		(end 73.35 86.1695)
+		(start 107.975 68.7)
+		(end 107.975 68.725)
 		(width 0.6)
 		(layer "In1.Cu")
@@
 	)
 	(segment
-		(start 73.35 93.98)
+		(start 73.35 95.93)
 		(end 73.35 112.12)
 		(width 0.6)
@@
 	)
 	(segment
-		(start 73.35 84.11)
-		(end 73.35 86.1695)
-		(width 0.6)
-		(layer "In1.Cu")
-		(net 25)
-	)
-	(segment
 		(start 85.84 84.07)
 		(end 84.324 84.07)
@@
 	)
 	(segment
-		(start 72.798 70.198)
-		(end 72.798 68.137)
-		(width 0.6)
-		(layer "In1.Cu")
-		(net 25)
-	)
-	(segment
-		(start 73.35 92.9715)
-		(end 71.4375 91.059)
+		(start 73.3405 66.4845)
+		(end 72.798 67.027)
 		(width 0.6)
 		(layer "In1.Cu")
@@
 	)
 	(segment
-		(start 73.35 70.85)
-		(end 73.35 84.11)
+		(start 75.79 93.49)
+		(end 73.35 95.93)
 		(width 0.6)
 		(layer "In1.Cu")
@@
 	)
 	(segment
-		(start 72.798 68.137)
-		(end 72.798 67.027)
+		(start 72.798 67.027)
+		(end 72.798 70.198)
 		(width 0.6)
 		(layer "In1.Cu")
@@
 	)
 	(segment
-		(start 73.35 93.98)
-		(end 73.35 92.9715)
-		(width 0.6)
-		(layer "In1.Cu")
-		(net 25)
-	)
-	(segment
 		(start 91.205 125.535)
 		(end 91.205 133.295)
@@
 	)
 	(via
-		(at 66.4845 132.2705)
+		(at 82.423 130.7465)
 		(size 0.8)
 		(drill 0.4)
@@
 	)
 	(via
-		(at 82.423 130.7465)
+		(at 66.4845 132.2705)
 		(size 0.8)
 		(drill 0.4)
@@
 	)
 	(segment
-		(start 60.82 134.84)
-		(end 64.99 134.84)
+		(start 84.091031 129.684031)
+		(end 67.802405 129.684031)
 		(width 0.25)
 		(layer "B.Cu")
@@
 	)
 	(segment
-		(start 84.8995 130.4925)
-		(end 84.091031 129.684031)
+		(start 64.737528 132.751)
+		(end 65.660046 131.828482)
 		(width 0.25)
 		(layer "B.Cu")
@@
 	)
 	(segment
-		(start 67.802405 129.684031)
-		(end 65.659 131.827436)
+		(start 60.82 134.84)
+		(end 62.909 132.751)
 		(width 0.25)
 		(layer "B.Cu")
@@
 	)
 	(segment
-		(start 84.091031 129.684031)
-		(end 67.802405 129.684031)
+		(start 62.909 132.751)
+		(end 64.737528 132.751)
 		(width 0.25)
 		(layer "B.Cu")
@@
 	)
 	(segment
-		(start 65.659 131.827436)
-		(end 65.659 134.171)
+		(start 84.8995 130.4925)
+		(end 84.091031 129.684031)
 		(width 0.25)
 		(layer "B.Cu")
@@
 	)
 	(segment
-		(start 65.659 134.171)
-		(end 64.99 134.84)
+		(start 67.802405 129.684031)
+		(end 65.659 131.827436)
 		(width 0.25)
 		(layer "B.Cu")
@@
 	(segment
 		(start 80.9575 79.9625)
-		(end 80.9575 89.5985)
+		(end 80.9575 91.53)
 		(width 0.4)
 		(layer "F.Cu")
@@
 	)
 	(segment
+		(start 77.089 103.632)
+		(end 77.089 102.4255)
+		(width 0.25)
+		(layer "In1.Cu")
+		(net 82)
+	)
+	(segment
 		(start 77.089 103.759)
 		(end 77.089 108.585)
@@
 	)
 	(segment
-		(start 80.9575 89.5985)
-		(end 79.629 90.927)
+		(start 79.629 92.8585)
+		(end 80.9575 91.53)
 		(width 0.25)
 		(layer "In1.Cu")
@@
 	(segment
 		(start 79.629 99.8855)
-		(end 79.629 91.3765)
+		(end 79.629 92.8585)
 		(width 0.25)
 		(layer "In1.Cu")
@@
 		(width 0.25)
 		(layer "In1.Cu")
-		(net 82)
-	)
-	(segment
-		(start 79.629 90.927)
-		(end 79.629 91.3765)
-		(width 0.25)
-		(layer "In1.Cu")
-		(net 82)
-	)
-	(segment
-		(start 77.089 103.632)
-		(end 77.089 102.4255)
-		(width 0.25)
-		(layer "In1.Cu")
