File: Kicad/Chat_Cartridge_V1.5/ZX_Cartridge.kicad_pcb (KiCad board)
At the start: 4 copper layers, 85.7 x 71.3 mm, 30 parts, among them Q1 2N7002, Q2 2N7002, Q3 AO3401A, SW1 SW_Push, U10 4075, U2 74LS165, U3 mini_esp32, U4 74HC595, U5 5v module (hx1314G based), U6 TXS0108EPW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

Commit message: kicad
Parts:
- moved R2 29.4 mm to (103.5, 82.5)
Routing:
- net Net-(U3-IO_13/TCK): track 3.51 -> 34.1 mm
- net IO2_L: track 44.5 -> 14.9 mm
- net D3: track 85.1 -> 94.7 mm
- net Net-(D2-K): track 37.9 -> 35.7 mm
- net RCLK_H: track 25.1 -> 26.6 mm
- net RomCE: track 68.5 -> 67.2 mm, vias 2 -> 1
- net A0: track 90.5 -> 89.4 mm, vias 3 -> 2
- net 12V: track 49.5 -> 48.6 mm
- net IO2_H: track 22.7 -> 22.0 mm
- net GND: vias 24 -> 29
